Commit message: Integrate canonical RUKA2 geometry

File: ruka2_control/ros2_control/ruka2.ros2_control.xacro (robot description, xacro)
@@ -19,4 +19,12 @@
         </joint>
       </xacro:macro>
+      <xacro:macro name="ruka2_mock_passive_joint" params="joint_name">
+        <joint name="${joint_name}">
+          <state_interface name="position">
+            <param name="initial_value">0.0</param>
+          </state_interface>
+          <state_interface name="velocity"/>
+        </joint>
+      </xacro:macro>
       <xacro:ruka2_mock_joint joint_name="joint_1"/>
       <xacro:ruka2_mock_joint joint_name="joint_2"/>
@@ -25,4 +33,6 @@
       <xacro:ruka2_mock_joint joint_name="joint_5"/>
       <xacro:ruka2_mock_joint joint_name="joint_6"/>
+      <xacro:ruka2_mock_passive_joint joint_name="link_hand_cyl__first_fin"/>
+      <xacro:ruka2_mock_passive_joint joint_name="link_hand_cyl__second_fin"/>
     </ros2_control>
   </xacro:macro>

File: ruka2_control/urdf/ruka2_control.urdf.xacro (robot description, xacro)
@@ -1,5 +1,4 @@
 <?xml version="1.0"?>
 <robot xmlns:xacro="http://www.ros.org/wiki/xacro" name="ruka2">
-  <!-- TEMPORARY DUMMY composition used only for software integration. -->
   <xacro:include filename="$(find ruka2_description)/urdf/ruka2_macro.urdf.xacro"/>
   <xacro:include filename="$(find ruka2_control)/ros2_control/ruka2.ros2_control.xacro"/>
@@ -7,5 +6,5 @@
     name="initial_positions_file"
     default="$(find ruka2_control)/config/initial_positions.yaml"/>
-  <xacro:ruka2_dummy/>
+  <xacro:ruka2_model/>
   <xacro:ruka2_mock_ros2_control
     name="Ruka2MockSystem"

File: ruka2_description/urdf/ruka2.urdf.xacro (robot description, xacro)
@@ -2,4 +2,4 @@
 <robot xmlns:xacro="http://www.ros.org/wiki/xacro" name="ruka2">
   <xacro:include filename="$(find ruka2_description)/urdf/ruka2_macro.urdf.xacro"/>
-  <xacro:ruka2_dummy/>
+  <xacro:ruka2_model/>
 </robot>

File: ruka2_description/urdf/ruka2_macro.urdf.xacro (robot description, xacro)
@@ -2,92 +2,674 @@
 <robot xmlns:xacro="http://www.ros.org/wiki/xacro">
   <!--
-    TEMPORARY DUMMY MODEL.
-    Dimensions, masses, axes, limits, and transforms are only for software
-    integration tests and must not be used for hardware commissioning.
+    Canonical RUKA2 geometry imported from the delivered ruka.urdf baseline.
+    The six arm axes are normalized to joint_1...joint_6. The gripper links
+    remain in the description for future integration but are not controlled.
   -->
-  <xacro:macro name="ruka2_dummy_link" params="name length:=0.16 radius:=0.035 color:='0.30 0.55 0.85 1'">
-    <link name="${name}">
-      <inertial>
-        <origin xyz="${length / 2.0} 0 0" rpy="0 0 0"/>
-        <mass value="0.25"/>
-        <inertia ixx="0.0002" ixy="0" ixz="0" iyy="0.0007" iyz="0" izz="0.0007"/>
-      </inertial>
-      <visual>
-        <origin xyz="${length / 2.0} 0 0" rpy="0 1.57079632679 0"/>
-        <geometry><cylinder radius="${radius}" length="${length}"/></geometry>
-        <material name="${name}_material"><color rgba="${color}"/></material>
-      </visual>
-      <collision>
-        <origin xyz="${length / 2.0} 0 0" rpy="0 1.57079632679 0"/>
-        <geometry><cylinder radius="${radius}" length="${length}"/></geometry>
-      </collision>
-    </link>
-  </xacro:macro>
-  <xacro:macro name="ruka2_dummy" params="prefix:=''">
-    <link name="${prefix}base_link">
-      <visual>
-        <origin xyz="0 0 0.04"/>
-        <geometry><cylinder radius="0.08" length="0.08"/></geometry>
-        <material name="dummy_base"><color rgba="0.20 0.22 0.25 1"/></material>
-      </visual>
-      <collision>
-        <origin xyz="0 0 0.04"/>
-        <geometry><cylinder radius="0.08" length="0.08"/></geometry>
-      </collision>
-    </link>
-    <xacro:ruka2_dummy_link name="${prefix}link_1" length="0.18"/>
-    <xacro:ruka2_dummy_link name="${prefix}link_2" length="0.22"/>
-    <xacro:ruka2_dummy_link name="${prefix}link_3" length="0.20"/>
-    <xacro:ruka2_dummy_link name="${prefix}link_4" length="0.15" radius="0.03"/>
-    <xacro:ruka2_dummy_link name="${prefix}link_5" length="0.12" radius="0.028"/>
-    <xacro:ruka2_dummy_link name="${prefix}link_6" length="0.10" radius="0.025"/>
-    <joint name="${prefix}joint_1" type="revolute">
-      <origin xyz="0 0 0.08" rpy="0 0 0"/>
-      <parent link="${prefix}base_link"/>
-      <child link="${prefix}link_1"/>
-      <axis xyz="0 0 1"/>
-      <limit lower="-3.14159" upper="3.14159" effort="20" velocity="1.0"/>
-    </joint>
-    <joint name="${prefix}joint_2" type="revolute">
-      <origin xyz="0.18 0 0" rpy="0 0 0"/>
-      <parent link="${prefix}link_1"/>
-      <child link="${prefix}link_2"/>
-      <axis xyz="0 1 0"/>
-      <limit lower="-2.6" upper="2.6" effort="20" velocity="1.0"/>
-    </joint>
-    <joint name="${prefix}joint_3" type="revolute">
-      <origin xyz="0.22 0 0" rpy="0 0 0"/>
-      <parent link="${prefix}link_2"/>
-      <child link="${prefix}link_3"/>
-      <axis xyz="0 1 0"/>
-      <limit lower="-2.8" upper="2.8" effort="20" velocity="1.0"/>
-    </joint>
-    <joint name="${prefix}joint_4" type="revolute">
-      <origin xyz="0.20 0 0" rpy="0 0 0"/>
-      <parent link="${prefix}link_3"/>
-      <child link="${prefix}link_4"/>
-      <axis xyz="1 0 0"/>
-      <limit lower="-3.14159" upper="3.14159" effort="10" velocity="1.5"/>
-    </joint>
-    <joint name="${prefix}joint_5" type="revolute">
-      <origin xyz="0.15 0 0" rpy="0 0 0"/>
-      <parent link="${prefix}link_4"/>
-      <child link="${prefix}link_5"/>
-      <axis xyz="0 1 0"/>
-      <limit lower="-2.6" upper="2.6" effort="10" velocity="1.5"/>
-    </joint>
-    <joint name="${prefix}joint_6" type="revolute">
-      <origin xyz="0.12 0 0" rpy="0 0 0"/>
-      <parent link="${prefix}link_5"/>
-      <child link="${prefix}link_6"/>
-      <axis xyz="1 0 0"/>
-      <limit lower="-3.14159" upper="3.14159" effort="5" velocity="2.0"/>
-    </joint>
-    <link name="${prefix}tool0"/>
-    <joint name="${prefix}tool0_joint" type="fixed">
-      <origin xyz="0.10 0 0" rpy="0 0 0"/>
-      <parent link="${prefix}link_6"/>
-      <child link="${prefix}tool0"/>
-    </joint>
+  <xacro:macro name="ruka2_model" params="">
+    <material name="white">
+            <color rgba="1 1 1 1"/>
+        </material>
+        <material name="red">
+            <color rgba="1 0 0 1"/>
+        </material>
+        <material name="blue">
+            <color rgba="0 0 1 1"/>
+        </material>
+        <link name="base_link">
+            <visual>
+              <origin rpy="0 0 0" xyz="0 0 0.025" />
+              <geometry>
+                <cylinder radius="0.09" length="0.05" />
+              </geometry>
+            <material name="white"/>
+            </visual>
+            <collision>
+                <origin rpy="0 0 0" xyz="0 0 0.025" />
+              <geometry>
+                <cylinder radius="0.09" length="0.05" />
+              </geometry>
+              </collision>
+        </link>
+        <joint name="joint_1" type="revolute">
+            <axis xyz="0 0 1"/>
+            <safety_controller k_position="100.0" k_velocity="200.0" soft_lower_limit="-2.908" soft_upper_limit="2.908" />
+            <limit effort="1000.0" lower="-2.96" upper="2.96" velocity="0.75"/>
+            <origin rpy="0 0 0" xyz="0 0 0.05"/>
+            <parent link="base_link"/>
+            <child link="link_01"/>
+        </joint>
+        <link name="link_01">
+            <visual>
+                <origin rpy="0 0 0" xyz="0 0 0.016" />
+                <geometry>
+                    <cylinder radius="0.047" length="0.032" />
+                </geometry>
+                <material name="white"/>
+            </visual>
+            <collision>
+                <origin rpy="0 0 0" xyz="0 0 0.016" />
+                <geometry>
+                    <cylinder radius="0.047" length="0.032" />
+                </geometry>
+              </collision>
+            <visual>
+                <origin rpy="0 0 0" xyz="-0.0365 0 0.085" />
+                <geometry>
+                    <box size ="0.173 0.148 0.106"/>
+                </geometry>
+            </visual>
+            <collision>
+               <origin rpy="0 0 0" xyz="-0.0365 0 0.085" />
+                <geometry>
+                    <box size ="0.173 0.148 0.106"/>
+                </geometry>
+              </collision>
+        </link>
+        <joint name="link_01__link_01_red" type="fixed">
+            <origin rpy="0 0 0" xyz="0.017 0 0"/>
+            <parent link="link_01"/>
+            <child link="link_01_red"/>
+        </joint>
+        <link name="link_01_red">
+            <visual>
+                <origin rpy="0 0 0" xyz="0 0.088 0.1165" />
+                <geometry>
+                    <box size="0.08 0.028 0.145"/>
+                </geometry>
+                <material name="red"/>
+            </visual>
+            <collision>
+                <origin rpy="0 0 0" xyz="0 0.088 0.1165" />
+                <geometry>
+                    <box size="0.08 0.028 0.145"/>
+                </geometry>
+              </collision>
+            <visual>
+                <origin rpy="0 0 0" xyz="0 -0.088 0.1165" />
+                <geometry>
+                    <box size="0.08 0.028 0.145"/>
+                </geometry>
+            </visual>
+            <collision>
+                <origin rpy="0 0 0" xyz="0 -0.088 0.1165" />
+                <geometry>
+                    <box size="0.08 0.028 0.145"/>
+                </geometry>
+              </collision>
+            <visual>
+                <origin rpy="1.57 0 0" xyz="0 -0.088 0.189" />
+                <geometry>
+                    <cylinder radius="0.04" length="0.028"/>
+                </geometry>
+            </visual>
+            <collision>
+               <origin rpy="1.57 0 0" xyz="0 -0.088 0.189" />
+                <geometry>
+                    <cylinder radius="0.04" length="0.028"/>
+                </geometry>
+              </collision>
+            <visual>
+                <origin rpy="1.57 0 0" xyz="0 0.088 0.189" />
+                <geometry>
+                    <cylinder radius="0.04" length="0.028"/>
+                </geometry>
+            </visual>
+            <collision>
+               <origin rpy="1.57 0 0" xyz="0 0.088 0.189" />
+                <geometry>
+                    <cylinder radius="0.04" length="0.028"/>
+                </geometry>
+              </collision>
+        </link>
+        <joint name="joint_2" type="revolute">
+            <axis xyz="0 0 1"/>
+            <!-- <safety_controller k_position="100.0" k_velocity="40.0" soft_lower_limit="-3.518" soft_upper_limit="-0.052" /> -->
+            <limit effort="1000.0" lower="-3.57" upper="0.05" velocity="0.6"/>
+            <origin rpy="1.57 -1.57 0" xyz="0.017 0 0.189"/>   <!-- origin rpy="1.57 0 0"-->
+            <parent link="link_01"/>
+            <child link="link_02"/>
+        </joint>
+        <link name="link_02">
+            <visual>
+                <origin rpy="0 0 0" xyz="0 0 0" />
+                <geometry>
+                    <cylinder radius="0.038" length="0.148"/>
+                </geometry>
+                <material name="white"/>
+            </visual>
+            <collision>
+                 <origin rpy="0 0 0" xyz="0 0 0" />
+                <geometry>
+                    <cylinder radius="0.038" length="0.148"/>
+                </geometry>
+              </collision>
+            <visual>
+                <origin rpy="0 0 0" xyz="0 0.06775 0" />
+                <geometry>
+                    <box size ="0.076 0.1355 0.116"/>
+                </geometry>
+                <material name="white"/>
+            </visual>
+            <collision>
+              <origin rpy="0 0 0" xyz="0 0.06775 0" />
+                <geometry>
+                    <box size ="0.076 0.1355 0.116"/>
+                </geometry>
+              </collision>
+            <visual>
+                <origin rpy="0 1.57 0" xyz="0 0.14 0.055" />
+                <geometry>
+                    <box size ="0.006 0.28 0.076"/>
+                </geometry>
+                <material name="white"/>
+            </visual>
+            <collision>
+                <origin rpy="0 1.57 0" xyz="0 0.14 0.055" />
+                <geometry>
+                    <box size ="0.006 0.28 0.076"/>
+                </geometry>
+              </collision>
+            <visual>
+                <origin rpy="0 1.57 0" xyz="0 0.14 -0.055" />
+                <geometry>
+                    <box size ="0.006 0.28 0.076"/>
+                </geometry>
+                <material name="white"/>
+            </visual>
+            <collision>
+                <origin rpy="0 1.57 0" xyz="0 0.14 -0.055" />
+                <geometry>
+                    <box size ="0.006 0.28 0.076"/>
+                </geometry>
+              </collision>
+            <visual>
+                <origin rpy="0 0 0" xyz="0 0.28 -0.055" />
+                <geometry>
+                    <cylinder radius="0.038" length="0.006"/>
+                </geometry>
+                <material name="white"/>
+            </visual>
+            <collision>
+                <origin rpy="0 0 0" xyz="0 0.28 -0.055" />
+                <geometry>
+                    <cylinder radius="0.038" length="0.006"/>
+                </geometry>
+              </collision>
+            <visual>
+                <origin rpy="0 0 0" xyz="0 0.28 0.055" />
+                <geometry>
+                    <cylinder radius="0.038" length="0.006"/>
+                </geometry>
+                <material name="white"/>
+            </visual>
+            <collision>
+                <origin rpy="0 0 0" xyz="0 0.28 0.055" />
+                <geometry>
+                    <cylinder radius="0.038" length="0.006"/>
+                </geometry>
+              </collision>
+        </link>
+        <joint name="link_02__link_02_red" type="fixed">
+            <origin rpy="0 0 0" xyz="0 0.181 0"/>
+            <parent link="link_02"/>
+            <child link="link_02_red"/>
+        </joint>
+        <link name="link_02_red">
+            <visual>
+                <origin rpy="0 0 0" xyz="0 0 0.069" />
+                <geometry>
+                    <box size="0.076 0.198 0.027"/>
+                </geometry>
+                <material name="red"/>
+            </visual>
+            <collision>
+                <origin rpy="0 0 0" xyz="0 0 0.069" />
+                <geometry>
+                    <box size="0.076 0.198 0.027"/>
+                </geometry>
+              </collision>
+            <visual>
+                <origin rpy="0 0 0" xyz="0 0 -0.069" />
+                <geometry>
+                    <box size="0.076 0.198 0.027"/>
+                </geometry>
+            </visual>
+            <collision>
+                <origin rpy="0 0 0" xyz="0 0 -0.069" />
+                <geometry>
+                    <box size="0.076 0.198 0.027"/>
+                </geometry>
+              </collision>
+            <visual>
+                <origin rpy="0 0 0" xyz="0 -0.099 0.069" />
+                <geometry>
+                    <cylinder radius="0.038" length="0.027"/>
+                </geometry>
+            </visual>
+            <collision>
+                <origin rpy="0 0 0" xyz="0 -0.099 0.069" />
+                <geometry>
+                    <cylinder radius="0.038" length="0.027"/>
+                </geometry>
+              </collision>
+            <visual>
+                <origin rpy="0 0 0" xyz="0 0.099 0.069" />
+                <geometry>
+                    <cylinder radius="0.038" length="0.027"/>
+                </geometry>
+            </visual>
+            <collision>
+                <origin rpy="0 0 0" xyz="0 0.099 0.069" />
+                <geometry>
+                    <cylinder radius="0.038" length="0.027"/>
+                </geometry>
+              </collision>
+            <visual>
+                <origin rpy="0 0 0" xyz="0 -0.099 -0.069" />
+                <geometry>
+                    <cylinder radius="0.038" length="0.027"/>
+                </geometry>
+            </visual>
+            <collision>
+                <origin rpy="0 0 0" xyz="0 -0.099 -0.069" />
+                <geometry>
+                    <cylinder radius="0.038" length="0.027"/>
+                </geometry>
+              </collision>
+            <visual>
+                <origin rpy="0 0 0" xyz="0 0.099 -0.069" />
+                <geometry>
+                    <cylinder radius="0.038" length="0.027"/>
+                </geometry>
+            </visual>
+            <collision>
+                 <origin rpy="0 0 0" xyz="0 0.099 -0.069" />
+                <geometry>
+                    <cylinder radius="0.038" length="0.027"/>
+                </geometry>
+              </collision>
+        </link>
+        <joint name="joint_3" type="revolute">
+            <axis xyz="0 0 1"/>
+            <!-- <safety_controller k_position="100.0" k_velocity="40.0" soft_lower_limit="0.067" soft_upper_limit="5.178" /> -->
+            <limit effort="1000.0" lower="-0.035" upper="5.23" velocity="0.75"/>
+            <origin rpy="0 0 0.0175" xyz="0 0.28 0"/>
+            <!-- !!!!!!!!!!!!!!!!!!!!! /> -->
+            <parent link="link_02"/>
+            <child link="link_03"/>
+        </joint>
+        <link name="link_03">
+            <visual>
+                <origin rpy="0 0 0" xyz="0 0 0" />
+                <geometry>
+                    <cylinder radius="0.019" length="0.104" />
+                </geometry>
+                <material name="white"/>
+            </visual>
+            <collision>
+                <origin rpy="0 0 0" xyz="0 0 0" />
+                <geometry>
+                    <cylinder radius="0.019" length="0.104" />
+                </geometry>
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
Commit message: Add real RUKA2 ros2_control hardware interface

File: ruka2_control/ros2_control/ruka2.ros2_control.xacro (robot description, xacro)
@@ -1,16 +1,36 @@
 <?xml version="1.0"?>
 <robot xmlns:xacro="http://www.ros.org/wiki/xacro">
-  <xacro:macro name="ruka2_mock_ros2_control" params="name initial_positions_file">
+  <xacro:macro
+    name="ruka2_ros2_control"
+    params="name initial_positions_file use_mock_hardware:=true can_interface:=vcan1.0 node_id:=100 queue_length:=1000 feedback_timeout:=0.25 heartbeat_timeout:=2.5 activation_timeout:=5.0 startup_grace:=1.0 require_all_joints_on_activate:=true">
     <xacro:property
       name="initial_positions"
       value="${xacro.load_yaml(initial_positions_file)['initial_positions']}"/>
+    <xacro:property
+      name="use_mock_hardware_bool"
+      value="${str(use_mock_hardware).lower() in ['true', '1', 'yes']}"/>
     <ros2_control name="${name}" type="system">
       <hardware>
-        <plugin>mock_components/GenericSystem</plugin>
-        <param name="calculate_dynamics">false</param>
+        <xacro:if value="${use_mock_hardware_bool}">
+          <plugin>mock_components/GenericSystem</plugin>
+          <param name="calculate_dynamics">false</param>
+        </xacro:if>
+        <xacro:unless value="${use_mock_hardware_bool}">
+          <plugin>ruka2_control/Ruka2System</plugin>
+          <param name="can_interface">${can_interface}</param>
+          <param name="node_id">${node_id}</param>
+          <param name="queue_length">${queue_length}</param>
+          <param name="feedback_timeout">${feedback_timeout}</param>
+          <param name="heartbeat_timeout">${heartbeat_timeout}</param>
+          <param name="activation_timeout">${activation_timeout}</param>
+          <param name="startup_grace">${startup_grace}</param>
+          <param name="maximum_servo_velocity">0.1</param>
+          <param name="require_all_joints_on_activate">${require_all_joints_on_activate}</param>
+        </xacro:unless>
       </hardware>
-      <xacro:macro name="ruka2_mock_joint" params="joint_name">
+      <xacro:macro name="ruka2_arm_joint" params="joint_name">
         <joint name="${joint_name}">
           <command_interface name="position"/>
+          <command_interface name="velocity"/>
           <state_interface name="position">
             <param name="initial_value">${initial_positions[joint_name]}</param>
@@ -27,12 +47,14 @@
         </joint>
       </xacro:macro>
-      <xacro:ruka2_mock_joint joint_name="joint_1"/>
-      <xacro:ruka2_mock_joint joint_name="joint_2"/>
-      <xacro:ruka2_mock_joint joint_name="joint_3"/>
-      <xacro:ruka2_mock_joint joint_name="joint_4"/>
-      <xacro:ruka2_mock_joint joint_name="joint_5"/>
-      <xacro:ruka2_mock_joint joint_name="joint_6"/>
-      <xacro:ruka2_mock_passive_joint joint_name="link_hand_cyl__first_fin"/>
-      <xacro:ruka2_mock_passive_joint joint_name="link_hand_cyl__second_fin"/>
+      <xacro:ruka2_arm_joint joint_name="joint_1"/>
+      <xacro:ruka2_arm_joint joint_name="joint_2"/>
+      <xacro:ruka2_arm_joint joint_name="joint_3"/>
+      <xacro:ruka2_arm_joint joint_name="joint_4"/>
+      <xacro:ruka2_arm_joint joint_name="joint_5"/>
+      <xacro:ruka2_arm_joint joint_name="joint_6"/>
+      <xacro:if value="${use_mock_hardware_bool}">
+        <xacro:ruka2_mock_passive_joint joint_name="link_hand_cyl__first_fin"/>
+        <xacro:ruka2_mock_passive_joint joint_name="link_hand_cyl__second_fin"/>
+      </xacro:if>
     </ros2_control>
   </xacro:macro>

File: ruka2_control/urdf/ruka2_control.urdf.xacro (robot description, xacro)
@@ -6,7 +6,25 @@
     name="initial_positions_file"
     default="$(find ruka2_control)/config/initial_positions.yaml"/>
+  <xacro:arg name="use_mock_hardware" default="true"/>
+  <xacro:arg name="can_interface" default="vcan1.0"/>
+  <xacro:arg name="node_id" default="100"/>
+  <xacro:arg name="queue_length" default="1000"/>
+  <xacro:arg name="feedback_timeout" default="0.25"/>
+  <xacro:arg name="heartbeat_timeout" default="2.5"/>
+  <xacro:arg name="activation_timeout" default="5.0"/>
+  <xacro:arg name="startup_grace" default="1.0"/>
+  <xacro:arg name="require_all_joints_on_activate" default="true"/>
   <xacro:ruka2_model/>
-  <xacro:ruka2_mock_ros2_control
-    name="Ruka2MockSystem"
-    initial_positions_file="$(arg initial_positions_file)"/>
+  <xacro:ruka2_ros2_control
+    name="Ruka2System"
+    initial_positions_file="$(arg initial_positions_file)"
+    use_mock_hardware="$(arg use_mock_hardware)"
+    can_interface="$(arg can_interface)"
+    node_id="$(arg node_id)"
+    queue_length="$(arg queue_length)"
+    feedback_timeout="$(arg feedback_timeout)"
+    heartbeat_timeout="$(arg heartbeat_timeout)"
+    activation_timeout="$(arg activation_timeout)"
+    startup_grace="$(arg startup_grace)"
+    require_all_joints_on_activate="$(arg require_all_joints_on_activate)"/>
 </robot>
