Commit message: feat: add selectable grippers and refine MoveIt setup

File: ruka2_control/config/ruka2.ros2_control.xacro (robot description, xacro)
@@ -3,5 +3,5 @@
   <xacro:macro
     name="ruka2_ros2_control"
-    params="name initial_positions_file use_mock_hardware:=true can_interface:=vcan1.0 node_id:=100 queue_length:=1000 feedback_timeout:=0.25 heartbeat_timeout:=2.5 activation_timeout:=5.0 startup_grace:=1.0 require_all_joints_on_activate:=true">
+    params="name initial_positions_file use_mock_hardware:=true end_effector_type:=mechanical can_interface:=vcan1.0 node_id:=100 queue_length:=1000 feedback_timeout:=0.25 heartbeat_timeout:=2.5 activation_timeout:=5.0 startup_grace:=1.0 require_all_joints_on_activate:=true">
     <xacro:property
       name="initial_positions"
@@ -10,4 +10,7 @@
       name="use_mock_hardware_bool"
       value="${str(use_mock_hardware).lower() in ['true', '1', 'yes']}"/>
+    <xacro:property
+      name="use_mock_mechanical_gripper"
+      value="${use_mock_hardware_bool and str(end_effector_type).lower() == 'mechanical'}"/>
     <ros2_control name="${name}" type="system">
       <hardware>
@@ -47,4 +50,13 @@
         </joint>
       </xacro:macro>
+      <xacro:macro name="ruka2_mock_gripper_joint" params="joint_name">
+        <joint name="${joint_name}">
+          <command_interface name="position"/>
+          <state_interface name="position">
+            <param name="initial_value">0.0</param>
+          </state_interface>
+          <state_interface name="velocity"/>
+        </joint>
+      </xacro:macro>
       <xacro:ruka2_arm_joint joint_name="joint_1"/>
       <xacro:ruka2_arm_joint joint_name="joint_2"/>
@@ -54,5 +66,10 @@
       <xacro:ruka2_arm_joint joint_name="joint_6"/>
       <xacro:if value="${use_mock_hardware_bool}">
-        <xacro:ruka2_mock_passive_joint joint_name="link_hand_cyl__first_fin"/>
+        <xacro:if value="${use_mock_mechanical_gripper}">
+          <xacro:ruka2_mock_gripper_joint joint_name="link_hand_cyl__first_fin"/>
+        </xacro:if>
+        <xacro:unless value="${use_mock_mechanical_gripper}">
+          <xacro:ruka2_mock_passive_joint joint_name="link_hand_cyl__first_fin"/>
+        </xacro:unless>
         <xacro:ruka2_mock_passive_joint joint_name="link_hand_cyl__second_fin"/>
       </xacro:if>

File: ruka2_control/config/ruka2_control.urdf.xacro (robot description, xacro)
@@ -8,4 +8,5 @@
   <xacro:arg name="use_mock_hardware" default="true"/>
   <xacro:arg name="use_end_effector" default="true"/>
+  <xacro:arg name="end_effector_type" default="mechanical"/>
   <xacro:arg name="can_interface" default="vcan1.0"/>
   <xacro:arg name="node_id" default="100"/>
@@ -16,9 +17,12 @@
   <xacro:arg name="startup_grace" default="1.0"/>
   <xacro:arg name="require_all_joints_on_activate" default="true"/>
-  <xacro:ruka2_model use_end_effector="$(arg use_end_effector)"/>
+  <xacro:ruka2_model
+    use_end_effector="$(arg use_end_effector)"
+    end_effector_type="$(arg end_effector_type)"/>
   <xacro:ruka2_ros2_control
     name="Ruka2System"
     initial_positions_file="$(arg initial_positions_file)"
     use_mock_hardware="$(arg use_mock_hardware)"
+    end_effector_type="$(arg end_effector_type)"
     can_interface="$(arg can_interface)"
     node_id="$(arg node_id)"

File: ruka2_description/urdf/ruka2.urdf.xacro (robot description, xacro)
@@ -3,4 +3,7 @@
   <xacro:include filename="$(find ruka2_description)/urdf/ruka2_macro.urdf.xacro"/>
   <xacro:arg name="use_end_effector" default="true"/>
-  <xacro:ruka2_model use_end_effector="$(arg use_end_effector)"/>
+  <xacro:arg name="end_effector_type" default="mechanical"/>
+  <xacro:ruka2_model
+    use_end_effector="$(arg use_end_effector)"
+    end_effector_type="$(arg end_effector_type)"/>
 </robot>

File: ruka2_description/urdf/ruka2_macro.urdf.xacro (robot description, xacro)
@@ -2,12 +2,32 @@
 <robot xmlns:xacro="http://www.ros.org/wiki/xacro">
   <!--
-    Canonical RUKA2 geometry imported from the delivered ruka.urdf baseline.
-    The six arm axes are normalized to joint_1...joint_6. The gripper links
-    remain in the description for future integration but are not controlled.
+    Основная геометрическая модель RUKA2.
+    Шесть осей руки имеют имена joint_1...joint_6. Звенья захвата входят в
+    общее описание робота и готовы к интеграции с системой управления.
   -->
-  <xacro:macro name="ruka2_model" params="use_end_effector:=true">
+  <xacro:macro
+    name="ruka2_model"
+    params="use_end_effector:=true end_effector_type:=mechanical">
     <xacro:property
       name="use_end_effector_bool"
       value="${str(use_end_effector).lower() in ['true', '1', 'yes']}"/>
+    <xacro:property
+      name="end_effector_type_value"
+      value="${str(end_effector_type).lower()}"/>
+    <xacro:property
+      name="show_mechanical_end_effector"
+      value="${use_end_effector_bool and end_effector_type_value == 'mechanical'}"/>
+    <xacro:property
+      name="show_electromagnetic_end_effector"
+      value="${use_end_effector_bool and end_effector_type_value == 'electromagnetic'}"/>
+    <xacro:property
+      name="tool0_x"
+      value="${-0.0272404332 if show_electromagnetic_end_effector else 0.0}"/>
+    <xacro:property
+      name="tool0_z"
+      value="${0.0879375831 if show_electromagnetic_end_effector else (0.1162 if show_mechanical_end_effector else 0.0)}"/>
+    <xacro:property
+      name="tool0_pitch"
+      value="${-0.4363323130 if show_electromagnetic_end_effector else 0.0}"/>
     <material name="white">
             <color rgba="1 1 1 1"/>
@@ -19,4 +39,7 @@
             <color rgba="0 0 1 1"/>
         </material>
+        <material name="gray">
+            <color rgba="0.45 0.45 0.45 1"/>
+        </material>
         <link name="base_link">
             <visual>
@@ -512,6 +535,6 @@
         </joint>
         <link name="link_05">
-            <!-- Light body: 74 mm wide, 82 mm long and 100 mm high.
-                 The J5 axis is 30 mm above its lower face. -->
+            <!-- Светлый корпус: ширина 74 мм, длина 82 мм, высота 100 мм.
+                 Ось J5 расположена на 30 мм выше нижней плоскости. -->
             <visual>
                 <origin rpy="0 1.57 0" xyz="0.020 0 0" />
@@ -534,5 +557,5 @@
         </joint>
         <link name="link_05_red">
-            <!-- Front cover towards the gripper: 20 mm thick. -->
+            <!-- Передняя крышка со стороны захвата: толщина 20 мм. -->
             <visual>
                 <origin rpy="0 1.57 0" xyz="0.020 -0.051 0" />
@@ -548,5 +571,5 @@
                 </geometry>
             </collision>
-            <!-- Rear cover: 27 mm thick. -->
+            <!-- Задняя крышка: толщина 27 мм. -->
             <visual>
                 <origin rpy="0 1.57 0" xyz="0.020 0.0545 0" />
@@ -572,5 +595,5 @@
         </joint>
         <link name="link_06">
-            <!-- The distal face is the gripper mounting plane. -->
+            <!-- Торцевая плоскость используется для установки захвата. -->
             <visual>
                 <origin rpy="0 0 0" xyz="0 0 -0.0125" />
@@ -593,5 +616,5 @@
         </joint>
         <link name="link_hand_cyl">
-          <xacro:if value="${use_end_effector_bool}">
+          <xacro:if value="${show_mechanical_end_effector}">
             <inertial>
                 <mass value="0.01"/>
@@ -616,5 +639,35 @@
             </collision>
           </xacro:if>
-        </link>
+          <xacro:if value="${show_electromagnetic_end_effector}">
+            <!-- Между окончанием link_05 и краем STL оставлено 5 мм link_06. -->
+            <visual name="electromagnetic_gripper_visual">
+              <origin
+                rpy="0 0 -1.5707963268"
+                xyz="-0.02 -0.0150980395 -0.0162865356"/>
+              <geometry>
+                <mesh filename="package://ruka2_description/meshes/mag-gripper.stl"/>
+              </geometry>
+              <material name="gray"/>
+            </visual>
+            <collision name="electromagnetic_gripper_collision">
+              <origin
+                rpy="0 0 -1.5707963268"
+                xyz="-0.02 -0.0150980395 -0.0162865356"/>
+              <geometry>
+                <mesh filename="package://ruka2_description/meshes/mag-gripper.stl"/>
+              </geometry>
+            </collision>
+          </xacro:if>
+        </link>
+        <!-- Общая TCP MoveIt: между концами механических пальцев, на рабочей
+             плоскости магнита либо в link_06, если захват не выбран. -->
+        <joint name="link_06__tool0" type="fixed">
+            <origin
+              rpy="0 ${tool0_pitch} 0"
+              xyz="${tool0_x} 0 ${tool0_z}"/>
+            <parent link="link_06"/>
+            <child link="tool0"/>
+        </joint>
+        <link name="tool0"/>
         <joint name="link_hand_cyl__first_fin" type="prismatic">
             <parent link="link_hand_cyl"/>
@@ -625,5 +678,5 @@
         </joint>
         <link name="first_fin">
-          <xacro:if value="${use_end_effector_bool}">
+          <xacro:if value="${show_mechanical_end_effector}">
             <inertial>
                 <mass value="0.01"/>
@@ -655,7 +708,13 @@
             <axis xyz="0 0 1"/>
             <limit effort="20" lower="0.0" upper="0.01" velocity="0.2"/>
+            <!-- Оси суставов зеркальны, поэтому multiplier 1 перемещает пальцы
+                 на одинаковое расстояние в противоположных направлениях. -->
+            <mimic
+              joint="link_hand_cyl__first_fin"
+              multiplier="1.0"
+              offset="0.0"/>
         </joint>
         <link name="second_fin">
-          <xacro:if value="${use_end_effector_bool}">
+          <xacro:if value="${show_mechanical_end_effector}">
             <inertial>
                 <mass value="0.01"/>

File: ruka2_moveit_config/config/ruka2.urdf.xacro (robot description, xacro)
@@ -1,6 +1,6 @@
 <?xml version="1.0"?>
 <robot xmlns:xacro="http://www.ros.org/wiki/xacro" name="ruka2">
-  <!-- Keep MoveIt configuration self-contained while the canonical model stays
-       in ruka2_description and ros2_control stays in ruka2_control. -->
+  <!-- Конфигурация MoveIt остаётся самодостаточной, основная модель хранится в
+       ruka2_description, а настройки ros2_control — в ruka2_control. -->
   <xacro:include filename="$(find ruka2_control)/config/ruka2_control.urdf.xacro"/>
 </robot>
