Commit message: Streamline RUKA2 launch and MoveIt setup

File: ruka2_control/config/ruka2_control.urdf.xacro (robot description, xacro)
@@ -2,9 +2,10 @@
 <robot xmlns:xacro="http://www.ros.org/wiki/xacro" name="ruka2">
   <xacro:include filename="$(find ruka2_description)/urdf/ruka2_macro.urdf.xacro"/>
-  <xacro:include filename="$(find ruka2_control)/ros2_control/ruka2.ros2_control.xacro"/>
+  <xacro:include filename="$(find ruka2_control)/config/ruka2.ros2_control.xacro"/>
   <xacro:arg
     name="initial_positions_file"
     default="$(find ruka2_control)/config/initial_positions.yaml"/>
   <xacro:arg name="use_mock_hardware" default="true"/>
+  <xacro:arg name="use_end_effector" default="true"/>
   <xacro:arg name="can_interface" default="vcan1.0"/>
   <xacro:arg name="node_id" default="100"/>
@@ -15,5 +16,5 @@
   <xacro:arg name="startup_grace" default="1.0"/>
   <xacro:arg name="require_all_joints_on_activate" default="true"/>
-  <xacro:ruka2_model/>
+  <xacro:ruka2_model use_end_effector="$(arg use_end_effector)"/>
   <xacro:ruka2_ros2_control
     name="Ruka2System"

File: ruka2_description/urdf/ruka2.urdf.xacro (robot description, xacro)
@@ -2,4 +2,5 @@
 <robot xmlns:xacro="http://www.ros.org/wiki/xacro" name="ruka2">
   <xacro:include filename="$(find ruka2_description)/urdf/ruka2_macro.urdf.xacro"/>
-  <xacro:ruka2_model/>
+  <xacro:arg name="use_end_effector" default="true"/>
+  <xacro:ruka2_model use_end_effector="$(arg use_end_effector)"/>
 </robot>

File: ruka2_description/urdf/ruka2_macro.urdf.xacro (robot description, xacro)
@@ -6,5 +6,8 @@
     remain in the description for future integration but are not controlled.
   -->
-  <xacro:macro name="ruka2_model" params="">
+  <xacro:macro name="ruka2_model" params="use_end_effector:=true">
+    <xacro:property
+      name="use_end_effector_bool"
+      value="${str(use_end_effector).lower() in ['true', '1', 'yes']}"/>
     <material name="white">
             <color rgba="1 1 1 1"/>
@@ -590,4 +593,5 @@
         </joint>
         <link name="link_hand_cyl">
+          <xacro:if value="${use_end_effector_bool}">
             <inertial>
                 <mass value="0.01"/>
@@ -611,4 +615,5 @@
                 </geometry>
             </collision>
+          </xacro:if>
         </link>
         <joint name="link_hand_cyl__first_fin" type="prismatic">
@@ -620,4 +625,5 @@
         </joint>
         <link name="first_fin">
+          <xacro:if value="${use_end_effector_bool}">
             <inertial>
                 <mass value="0.01"/>
@@ -641,4 +647,5 @@
                 </geometry>
             </collision>
+          </xacro:if>
         </link>
         <joint name="link_hand_cyl__second_fin" type="prismatic">
@@ -650,4 +657,5 @@
         </joint>
         <link name="second_fin">
+          <xacro:if value="${use_end_effector_bool}">
             <inertial>
                 <mass value="0.01"/>
@@ -671,4 +679,5 @@
                 </geometry>
             </collision>
+          </xacro:if>
         </link>
   </xacro:macro>

Commit message: fix: align real robot model with calibrated joints

File: ruka2_control/config/ruka2_control.urdf.xacro (robot description, xacro)
@@ -19,5 +19,6 @@
   <xacro:ruka2_model
     use_end_effector="$(arg use_end_effector)"
-    end_effector_type="$(arg end_effector_type)"/>
+    end_effector_type="$(arg end_effector_type)"
+    enable_gripper_motion="$(arg use_mock_hardware)"/>
   <xacro:ruka2_ros2_control
     name="Ruka2System"

File: ruka2_description/urdf/ruka2.urdf.xacro (robot description, xacro)
@@ -4,6 +4,8 @@
   <xacro:arg name="use_end_effector" default="true"/>
   <xacro:arg name="end_effector_type" default="mechanical"/>
+  <xacro:arg name="enable_gripper_motion" default="true"/>
   <xacro:ruka2_model
     use_end_effector="$(arg use_end_effector)"
-    end_effector_type="$(arg end_effector_type)"/>
+    end_effector_type="$(arg end_effector_type)"
+    enable_gripper_motion="$(arg enable_gripper_motion)"/>
 </robot>

File: ruka2_description/urdf/ruka2_macro.urdf.xacro (robot description, xacro)
@@ -8,5 +8,5 @@
   <xacro:macro
     name="ruka2_model"
-    params="use_end_effector:=true end_effector_type:=mechanical">
+    params="use_end_effector:=true end_effector_type:=mechanical enable_gripper_motion:=true">
     <xacro:property
       name="use_end_effector_bool"
@@ -15,4 +15,7 @@
       name="end_effector_type_value"
       value="${str(end_effector_type).lower()}"/>
+    <xacro:property
+      name="enable_gripper_motion_bool"
+      value="${str(enable_gripper_motion).lower() in ['true', '1', 'yes']}"/>
     <xacro:property
       name="show_mechanical_end_effector"
@@ -59,6 +62,6 @@
         <joint name="joint_1" type="revolute">
             <axis xyz="0 0 1"/>
-            <safety_controller k_position="100.0" k_velocity="200.0" soft_lower_limit="-2.908" soft_upper_limit="2.908" />
-            <limit effort="1000.0" lower="-2.96" upper="2.96" velocity="0.75"/>
+            <safety_controller k_position="100.0" k_velocity="200.0" soft_lower_limit="-2.833300981" soft_upper_limit="2.833300981" />
+            <limit effort="1000.0" lower="-2.91" upper="2.91" velocity="0.75"/>
             <origin rpy="0 0 0" xyz="0 0 0.05"/>
             <parent link="base_link"/>
@@ -150,6 +153,6 @@
         <joint name="joint_2" type="revolute">
             <axis xyz="0 0 1"/>
-            <!-- <safety_controller k_position="100.0" k_velocity="40.0" soft_lower_limit="-3.518" soft_upper_limit="-0.052" /> -->
-            <limit effort="1000.0" lower="-3.57" upper="0.05" velocity="0.6"/>
+            <safety_controller k_position="100.0" k_velocity="40.0" soft_lower_limit="-3.293300981" soft_upper_limit="-0.056699019" />
+            <limit effort="1000.0" lower="-3.37" upper="0.02" velocity="0.6"/>
             <origin rpy="1.57 -1.57 0" xyz="0.017 0 0.189"/>   <!-- origin rpy="1.57 0 0"-->
             <parent link="link_01"/>
@@ -318,6 +321,6 @@
         <joint name="joint_3" type="revolute">
             <axis xyz="0 0 1"/>
-            <!-- <safety_controller k_position="100.0" k_velocity="40.0" soft_lower_limit="0.067" soft_upper_limit="5.178" /> -->
-            <limit effort="1000.0" lower="-0.035" upper="5.23" velocity="0.75"/>
+            <safety_controller k_position="100.0" k_velocity="40.0" soft_lower_limit="0.076699019" soft_upper_limit="5.033300981" />
+            <limit effort="1000.0" lower="0.0" upper="5.11" velocity="0.75"/>
             <origin rpy="0 0 0.0175" xyz="0 0.28 0"/>
             <!-- !!!!!!!!!!!!!!!!!!!!! /> -->
@@ -387,6 +390,6 @@
         <joint name="joint_4" type="revolute">
             <axis xyz="0 0 1"/>
-            <safety_controller k_position="100.0" k_velocity="40.0" soft_lower_limit="-2.818" soft_upper_limit="2.818" />
-            <limit effort="1000.0" lower="-2.87" upper="2.87" velocity="2.0"/>
+            <safety_controller k_position="100.0" k_velocity="40.0" soft_lower_limit="-2.343300981" soft_upper_limit="3.123300981" />
+            <limit effort="1000.0" lower="-2.42" upper="3.20" velocity="2.0"/>
             <origin rpy="1.57 0 0" xyz="0.072 0 0"/>
             <parent link="link_03"/>
@@ -528,6 +531,6 @@
         <joint name="joint_5" type="revolute">
             <axis xyz="0 0 1"/>
-            <safety_controller k_position="100.0" k_velocity="40.0" soft_lower_limit="-2.388" soft_upper_limit="2.388" />
-            <limit effort="1000.0" lower="-2.44" upper="2.44" velocity="2.5"/>
+            <safety_controller k_position="100.0" k_velocity="40.0" soft_lower_limit="-2.313300981" soft_upper_limit="2.313300981" />
+            <limit effort="1000.0" lower="-2.39" upper="2.39" velocity="2.5"/>
             <origin rpy="-1.57 0 0" xyz="0 0 0.264"/>
             <parent link="link_04"/>
@@ -588,6 +591,6 @@
         <joint name="joint_6" type="revolute">
             <axis xyz="0 0 1"/>
-            <safety_controller k_position="100.0" k_velocity="40.0" soft_lower_limit="-3.12" soft_upper_limit="3.12" />
-            <limit effort="1000.0" lower="-3.14" upper="3.14" velocity="6.0"/>
+            <safety_controller k_position="100.0" k_velocity="40.0" soft_lower_limit="-2.743300981" soft_upper_limit="2.763300981" />
+            <limit effort="1000.0" lower="-2.82" upper="2.84" velocity="6.0"/>
             <origin rpy="1.57 0 0" xyz="0 -0.086 0"/>
             <parent link="link_05"/>
@@ -670,10 +673,14 @@
         </joint>
         <link name="tool0"/>
-        <joint name="link_hand_cyl__first_fin" type="prismatic">
+        <joint
+          name="link_hand_cyl__first_fin"
+          type="${'prismatic' if enable_gripper_motion_bool else 'fixed'}">
             <parent link="link_hand_cyl"/>
             <child link="first_fin"/>
             <origin rpy="1.57 0 3.14" xyz="0 0.005 0.0642"/>
-            <axis xyz="0 0 1"/>
-            <limit effort="20" lower="0.0" upper="0.01" velocity="0.2"/>
+            <xacro:if value="${enable_gripper_motion_bool}">
+              <axis xyz="0 0 1"/>
+              <limit effort="20" lower="0.0" upper="0.01" velocity="0.2"/>
+            </xacro:if>
         </joint>
         <link name="first_fin">
@@ -702,16 +709,20 @@
           </xacro:if>
         </link>
-        <joint name="link_hand_cyl__second_fin" type="prismatic">
+        <joint
+          name="link_hand_cyl__second_fin"
+          type="${'prismatic' if enable_gripper_motion_bool else 'fixed'}">
             <parent link="link_hand_cyl"/>
             <child link="second_fin"/>
             <origin rpy="1.57 0 0" xyz="0 -0.005 0.0642"/>
-            <axis xyz="0 0 1"/>
-            <limit effort="20" lower="0.0" upper="0.01" velocity="0.2"/>
-            <!-- Оси суставов зеркальны, поэтому multiplier 1 перемещает пальцы
-                 на одинаковое расстояние в противоположных направлениях. -->
-            <mimic
-              joint="link_hand_cyl__first_fin"
-              multiplier="1.0"
-              offset="0.0"/>
+            <xacro:if value="${enable_gripper_motion_bool}">
+              <axis xyz="0 0 1"/>
+              <limit effort="20" lower="0.0" upper="0.01" velocity="0.2"/>
+              <!-- Оси суставов зеркальны, поэтому multiplier 1 перемещает пальцы
+                   на одинаковое расстояние в противоположных направлениях. -->
+              <mimic
+                joint="link_hand_cyl__first_fin"
+                multiplier="1.0"
+                offset="0.0"/>
+            </xacro:if>
         </joint>
         <link name="second_fin">
