Commit message: Limit joint 5 with mechanical gripper

File: ruka_spb/config/ruka.urdf (robot description, URDF)
Before this commit: robot ruka, 16 links, 15 joints
Joints:
- joint joint_5: limit lower=-2.39 upper=2.39 effort=1000.0 velocity=1.0 -> lower=-2.39 upper=${joint_5_upper_limit} effort=1000.0 velocity=1.0

File: ruka_spb/config/ruka.urdf.xacro (robot description, xacro)
@@ -24,4 +24,11 @@
     name="show_electromagnetic_end_effector"
     value="${selected_end_effector == 'electromagnetic'}"/>
+  <!-- The mechanical gripper limits positive J5 travel to avoid interference. -->
+  <xacro:property
+    name="joint_5_upper_limit"
+    value="${1.308996939 if show_mechanical_end_effector else 2.39}"/>
+  <xacro:property
+    name="joint_5_soft_upper_limit"
+    value="${1.308996939 if show_mechanical_end_effector else 2.313300981}"/>
   <xacro:property
     name="tool0_x"
